Commit message: Moved files around to clean up the workspace. RPi and esp files all in own folders at top level. Operator station scripts organised into packages.

File: scripts/gui/resource/fred-descr-v1.urdf (robot description, URDF)
Before this commit: robot FRED, 3 links, 2 joints
Links:
- link base_link: geometry visual box size=0.25 0.25 0.1
Joints:
- joint base_to_left_wheel: origin xyz=0.125 0 0 -> xyz=0 0 0
- joint base_to_right_wheel: origin xyz=0.125 0 0 -> xyz=0 0 0
